File: Power and ADC Module/Eagle/power_adc_module.brd (EAGLE design)
At the start: 63.5 x 48.3 mm, 11 parts

Commit message: Update: v1.1.0
Parts:
- added JP3: (no value), pinhead:1X15
- JP2: device pinhead:1X03 -> pinhead:1X15
- moved JP2 32.1 mm to (40.6, 11.4), turned to 0 degrees
- moved C3 7.41 mm to (30.5, 41.9), turned to 90 degrees
Connections:
- removed net 3V3: MODUL.J2.14
- removed net AREF: MODUL.J2.13
- removed net COM: MODUL.J1.4
- removed net VIN: MODUL.J2.1
- new net N$10: JP2.9, MODUL.J1.9
- new net N$11: JP2.10, MODUL.J1.10
- new net N$12: JP2.11, MODUL.J1.11
- new net N$13: JP2.12, MODUL.J1.12
- new net N$14: JP2.13, MODUL.J1.13
- new net N$15: JP2.14, MODUL.J1.14
- new net N$16: JP2.15, MODUL.J1.15
- new net N$17: JP3.1, MODUL.J2.1
- new net N$18: JP3.3, MODUL.J2.3
- new net N$19: JP3.5, MODUL.J2.5
- new net N$2: JP2.2, MODUL.J1.2
- new net N$20: JP3.6, MODUL.J2.6
- new net N$21: JP3.7, MODUL.J2.7
- new net N$22: JP3.8, MODUL.J2.8
- new net N$23: JP3.9, MODUL.J2.9
- new net N$24: JP3.10, MODUL.J2.10
- new net N$25: JP3.11, MODUL.J2.11
- new net N$26: JP3.15, MODUL.J2.15
- new net N$27: JP3.13, MODUL.J2.13
- new net N$28: JP3.14, MODUL.J2.14
- new net N$4: JP2.3, MODUL.J1.3
- new net N$5: JP2.4, MODUL.J1.4
- new net N$6: JP2.5, MODUL.J1.5
- new net N$7: JP2.6, MODUL.J1.6
- new net N$8: JP2.7, MODUL.J1.7
- new net N$9: JP2.8, MODUL.J1.8
- net GND: now also JP3.2; no longer JP2.2
- net IN5V: now also JP3.4; no longer JP2.1
- net N$3: now also JP2.1, MODUL.J1.1; no longer JP2.3, MODUL.J1.5
Routing:
- net N$3: track 55.9 -> 3.81 mm
- net GND: track 142.3 -> 105.2 mm
- net IN5V: track 48.3 -> 17.8 mm
- net N$9: track 0.00 -> 3.81 mm
- net N$8: track 0.00 -> 3.81 mm
- net N$7: track 0.00 -> 3.81 mm
- net N$6: track 0.00 -> 3.81 mm
- net N$5: track 0.00 -> 3.81 mm
- net N$4: track 0.00 -> 3.81 mm
- net N$2: track 0.00 -> 3.81 mm
- net N$16: track 0.00 -> 3.81 mm
- net N$15: track 0.00 -> 3.81 mm
- net N$14: track 0.00 -> 3.81 mm
- net N$13: track 0.00 -> 3.81 mm
- net N$12: track 0.00 -> 3.81 mm
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Other:
- board text added: "Open Plant Bioelectric Potential Measurement"
- board text added: "Power Module"
- board text added: "https://open-plant-bioelectric-potential-measurement.vercel.app"
- board text added: "v1.1.0"
