File: Signal Processing Module/Eagle/signal_processing_module.brd (EAGLE design)
At the start: 63.5 x 48.3 mm, 26 parts, among them IC1 LM324N, IC2 TL061P

Commit message: Update: v1.1.0
Parts:
- moved R10 0.25 mm to (33.0, 34.5)
- moved R14 0.25 mm to (35.6, 32.0)
Connections:
- removed net N$16: R13.2, R5.2
- net N$17: now also R13.2, R5.2
Routing:
- net GND: track 228.5 -> 211.4 mm
- net N$17: track 0.00 -> 5.09 mm
- net N$21: track 51.8 -> 56.0 mm
- net N$16: track 2.55 -> 0.00 mm
Other:
- board text added: "Open Plant Bioelectric Potential Measurement"
- board text added: "Signal Processing Module"
- board text added: "https://open-plant-bioelectric-potential-measurement.vercel.app"
- board text added: "v1.1.0"

Commit message: v1.1.1を更新
Parts:
- R16: value 50k -> 100k
- renumbered LED to LED+
Connections:
- net N$10 renamed OUT
- net N$17 renamed SIGNAL
Other:
- board text added: "v1.1.1"
- board text removed: "v1.1.0"
Changed lines of the file:
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@@
 <text x="7.62" y="2.54" size="1.016" layer="21">https://open-plant-bioelectric-potential-measurement.vercel.app</text>
 <text x="7.62" y="45.72" size="1.016" layer="21">Signal Processing Module</text>
-<text x="7.62" y="43.18" size="1.016" layer="21">v1.1.0</text>
+<text x="7.62" y="43.18" size="1.016" layer="21">v1.1.1</text>
 </plain>
 <attributes>
@@
 <attribute name="VALUE" x="56.3626" y="14.8844" size="0.9906" layer="27" ratio="10" rot="R90"/>
 </element>
-<element name="LED" library="led" library_urn="urn:adsk.eagle:library:259" package="LED3MM" package3d_urn="urn:adsk.eagle:package:15797/1" value="" x="58.42" y="11.43" smashed="yes" rot="R270">
+<element name="LED+" library="led" library_urn="urn:adsk.eagle:library:259" package="LED3MM" package3d_urn="urn:adsk.eagle:package:15797/1" value="" x="58.42" y="11.43" smashed="yes" rot="R270">
 <attribute name="NAME" x="58.801" y="9.525" size="1.27" layer="25" ratio="10" rot="R270"/>
 <attribute name="POPULARITY" value="97" x="58.42" y="11.43" size="1.778" layer="27" rot="R270" display="off"/>
@@
 <attribute name="VALUE" x="36.0426" y="30.3784" size="0.9906" layer="27" ratio="10" rot="R90"/>
 </element>
-<element name="R16" library="myparts" package="2CH_VR" value="50k" x="5.08" y="35.56" smashed="yes" rot="R180"/>
+<element name="R16" library="myparts" package="2CH_VR" value="100k" x="5.08" y="35.56" smashed="yes" rot="R180"/>
 <element name="R4" library="rcl" library_urn="urn:adsk.eagle:library:334" package="0204/7" package3d_urn="urn:adsk.eagle:package:23498/2" value="10k" x="38.1" y="11.43" smashed="yes" rot="R270">
 <attribute name="NAME" x="39.3954" y="13.97" size="0.9906" layer="25" ratio="10" rot="R270"/>
@@
 <contactref element="R13" pad="1"/>
 <contactref element="C4" pad="2"/>
-<contactref element="LED" pad="K"/>
+<contactref element="LED+" pad="K"/>
 <contactref element="JP1" pad="5"/>
 <wire x1="22.8534" y1="30.48" x2="22.86" y2="30.4866" width="1.27" layer="16"/>
@@
 <wire x1="38.1066" y1="43.18" x2="40.64" y2="43.18" width="1.27" layer="16"/>
 </signal>
-<signal name="N$10">
+<signal name="OUT">
 <contactref element="R12" pad="2"/>
 <contactref element="JP1" pad="1"/>
@@
 <signal name="N$11">
 <contactref element="R15" pad="1"/>
-<contactref element="LED" pad="A"/>
+<contactref element="LED+" pad="A"/>
 <wire x1="58.42" y1="12.7" x2="55.88" y2="12.7" width="1.27" layer="16"/>
 </signal>
@@
 <wire x1="50.8" y1="25.4066" x2="50.8" y2="27.94" width="1.27" layer="16"/>
 </signal>
-<signal name="N$17">
+<signal name="SIGNAL">
 <contactref element="R6" pad="1"/>
 <contactref element="R5" pad="2"/>
