File: Signal Processing Module/Eagle/signal_processing_module.sch (EAGLE design)
At the start: 26 parts, among them IC1 LM324N, IC2 TL061P

Commit message: Update: v1.1.0
Connections:
- removed net N$16: R13.2, R5.2
- net N$17: now also R13.2, R5.2
Other:
- moved on the sheet: R14
Changed lines of the file:
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@@
 </instance>
 <instance part="IC1" gate="P" x="96.52" y="66.04" smashed="yes"/>
-<instance part="R14" gate="G$1" x="99.06" y="55.88" smashed="yes">
-<attribute name="NAME" x="95.25" y="57.3786" size="1.778" layer="95"/>
-<attribute name="VALUE" x="100.33" y="57.658" size="1.778" layer="96"/>
+<instance part="R14" gate="G$1" x="104.14" y="55.88" smashed="yes">
+<attribute name="NAME" x="100.33" y="57.3786" size="1.778" layer="95"/>
+<attribute name="VALUE" x="105.41" y="57.658" size="1.778" layer="96"/>
 </instance>
 <instance part="R16" gate="G$2" x="88.9" y="43.18" smashed="yes" rot="R90">
@@
 <net name="RAW_SIGNAL" class="0">
 <segment>
-<wire x1="106.68" y1="66.04" x2="106.68" y2="55.88" width="0.1524" layer="91"/>
-<wire x1="104.14" y1="66.04" x2="106.68" y2="66.04" width="0.1524" layer="91"/>
-<junction x="106.68" y="66.04"/>
-<wire x1="106.68" y1="66.04" x2="109.22" y2="66.04" width="0.1524" layer="91"/>
+<wire x1="109.22" y1="66.04" x2="109.22" y2="55.88" width="0.1524" layer="91"/>
+<wire x1="104.14" y1="66.04" x2="109.22" y2="66.04" width="0.1524" layer="91"/>
+<junction x="109.22" y="66.04"/>
 <pinref part="R10" gate="G$1" pin="1"/>
 <pinref part="IC1" gate="B" pin="OUT"/>
-<wire x1="104.14" y1="55.88" x2="106.68" y2="55.88" width="0.1524" layer="91"/>
 <pinref part="R14" gate="G$1" pin="2"/>
 </segment>
@@
 <wire x1="88.9" y1="86.36" x2="91.44" y2="86.36" width="0.1524" layer="91"/>
 <pinref part="IC1" gate="A" pin="+IN"/>
-</segment>
-</net>
-<net name="N$16" class="0">
-<segment>
-<pinref part="R5" gate="G$1" pin="2"/>
-<wire x1="111.76" y1="129.54" x2="116.84" y2="129.54" width="0.1524" layer="91"/>
-<pinref part="R13" gate="G$1" pin="2"/>
-<wire x1="116.84" y1="124.46" x2="116.84" y2="129.54" width="0.1524" layer="91"/>
-<junction x="116.84" y="129.54"/>
-<wire x1="124.46" y1="129.54" x2="116.84" y2="129.54" width="0.1524" layer="91"/>
 </segment>
 </net>
@@
 <pinref part="IC1" gate="B" pin="-IN"/>
 <wire x1="88.9" y1="63.5" x2="88.9" y2="55.88" width="0.1524" layer="91"/>
-<wire x1="88.9" y1="55.88" x2="93.98" y2="55.88" width="0.1524" layer="91"/>
+<wire x1="88.9" y1="55.88" x2="99.06" y2="55.88" width="0.1524" layer="91"/>
 <pinref part="R14" gate="G$1" pin="1"/>
 <pinref part="R16" gate="G$2" pin="P$3"/>
@@
 <pinref part="R6" gate="G$1" pin="1"/>
 <wire x1="45.72" y1="68.58" x2="48.26" y2="68.58" width="0.1524" layer="91"/>
+<wire x1="45.72" y1="68.58" x2="45.72" y2="91.44" width="0.1524" layer="91"/>
+<wire x1="45.72" y1="91.44" x2="76.2" y2="91.44" width="0.1524" layer="91"/>
+<wire x1="76.2" y1="91.44" x2="76.2" y2="104.14" width="0.1524" layer="91"/>
+<wire x1="76.2" y1="104.14" x2="124.46" y2="104.14" width="0.1524" layer="91"/>
+<pinref part="R5" gate="G$1" pin="2"/>
+<wire x1="111.76" y1="129.54" x2="116.84" y2="129.54" width="0.1524" layer="91"/>
+<pinref part="R13" gate="G$1" pin="2"/>
+<wire x1="116.84" y1="124.46" x2="116.84" y2="129.54" width="0.1524" layer="91"/>
+<junction x="116.84" y="129.54"/>
+<wire x1="124.46" y1="129.54" x2="116.84" y2="129.54" width="0.1524" layer="91"/>
+<wire x1="124.46" y1="104.14" x2="124.46" y2="129.54" width="0.1524" layer="91"/>
 </segment>
 </net>
@@
 </sheet>
 </sheets>
+<errors>
+</errors>
 </schematic>
 </drawing>

Commit message: v1.1.1を更新
Parts:
- removed LED: (no value), led:LED3MM
- added LED+: (no value), led:LED3MM
- R16: value 50k -> 100k
Connections:
- net N$10 renamed OUT
- net N$17 renamed SIGNAL
- net GND: now also LED+.C, R16B.P$1, R16B.P$2; no longer LED.C, R16G$2.P$1, R16G$2.P$2
- net N$11: now also LED+.A; no longer LED.A
- net N$12: now also R16B.P$3; no longer R16G$2.P$3
Other:
- note removed: "RFノイズの除去"
- note removed: "R_f"
- moved on the sheet: C1, C2, C3, C4, C5, IC1A, IC1B, IC1C, IC1D, IC2, JP1, R1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
